File: 8086 Computer/8086 Computer.sch (KiCad schematic (older format))
At the start: 8 parts

Commit message: Started Work on Graphics
Parts:
- added U? (x3): 74LS161, symbol 74xx:74LS161
- added U?: 74LS30, symbol 74xx:74LS30
- added U?: 74LS00, symbol 74xx:74LS00
Connections:
- wire segments 14 -> 56
Changed lines of the file:
@@
 Text Label 6200 2300 1    50   ~ 0
 AL14
-Wire Bus Line
-	3150 800  3150 4750
-Wire Bus Line
-	3150 800  8450 800
-Wire Bus Line
-	4300 2000 10700 2000
-Wire Bus Line
-	6100 2200 10700 2200
-Wire Bus Line
-	10700 2000 14650 2000
 $Comp
 L power:GND #PWR?
@@
 	1    0    0    -1
 $EndComp
+$Comp
+L 74xx:74LS161 U?
+U 1 1 611A0ED4
+P 16300 7200
+F 0 "U?" H 16300 8181 50  0000 C CNN
+F 1 "74LS161" H 16300 8090 50  0000 C CNN
+F 2 "" H 16300 7200 50  0001 C CNN
+F 3 "http://www.ti.com/lit/gpn/sn74LS161" H 16300 7200 50  0001 C CNN
+	1    16300 7200
+	1    0    0    -1
+$EndComp
+$Comp
+L 74xx:74LS161 U?
+U 1 1 6119FD70
+P 16300 5350
+F 0 "U?" H 16300 6331 50  0000 C CNN
+F 1 "74LS161" H 16300 6240 50  0000 C CNN
+F 2 "" H 16300 5350 50  0001 C CNN
+F 3 "http://www.ti.com/lit/gpn/sn74LS161" H 16300 5350 50  0001 C CNN
+	1    16300 5350
+	1    0    0    -1
+$EndComp
+$Comp
+L 74xx:74LS30 U?
+U 1 1 611ABE17
+P 17900 3300
+F 0 "U?" H 17900 3825 50  0000 C CNN
+F 1 "74LS30" H 17900 3734 50  0000 C CNN
+F 2 "" H 17900 3300 50  0001 C CNN
+F 3 "http://www.ti.com/lit/gpn/sn74LS30" H 17900 3300 50  0001 C CNN
+	1    17900 3300
+	1    0    0    -1
+$EndComp
+Wire Wire Line
+	15800 3800 15600 3800
+Wire Wire Line
+	15600 7500 15800 7500
+Wire Wire Line
+	15800 7300 15350 7300
+Wire Wire Line
+	15350 7300 15350 7200
+Wire Wire Line
+	15800 7200 15350 7200
+Connection ~ 15350 7200
+Wire Wire Line
+	15800 3700 15350 3700
+Connection ~ 15350 3700
+Wire Wire Line
+	15350 3600 15800 3600
+$Comp
+L 74xx:74LS161 U?
+U 1 1 6119EEF4
+P 16300 3500
+F 0 "U?" H 16300 4481 50  0000 C CNN
+F 1 "74LS161" H 16300 4390 50  0000 C CNN
+F 2 "" H 16300 3500 50  0001 C CNN
+F 3 "http://www.ti.com/lit/gpn/sn74LS161" H 16300 3500 50  0001 C CNN
+	1    16300 3500
+	1    0    0    -1
+$EndComp
+Connection ~ 15350 3600
+Wire Wire Line
+	15350 3700 15350 3600
+Wire Wire Line
+	15350 3500 15350 3600
+Wire Wire Line
+	15800 3500 15350 3500
+Wire Wire Line
+	15350 3500 14300 3500
+Wire Wire Line
+	14300 3500 14300 3550
+Connection ~ 15350 3500
+$Comp
+L power:+5V #PWR?
+U 1 1 611C1BBC
+P 14300 3500
+F 0 "#PWR?" H 14300 3350 50  0001 C CNN
+F 1 "+5V" H 14315 3673 50  0000 C CNN
+F 2 "" H 14300 3500 50  0001 C CNN
+F 3 "" H 14300 3500 50  0001 C CNN
+	1    14300 3500
+	1    0    0    -1
+$EndComp
+Connection ~ 14300 3500
+Wire Wire Line
+	16800 3500 16800 4400
+Wire Wire Line
+	16800 4400 15500 4400
+Wire Wire Line
+	15500 4400 15500 5550
+Wire Wire Line
+	16800 5350 16800 6250
+Wire Wire Line
+	16800 6250 15500 6250
+Wire Wire Line
+	15500 6250 15500 7400
+Wire Wire Line
+	15500 7400 15800 7400
+Wire Wire Line
+	15700 7700 15800 7700
+Connection ~ 15350 5350
+Connection ~ 15350 5450
+Wire Wire Line
+	15350 5350 15350 3700
+Wire Wire Line
+	15350 5350 15350 5450
+Connection ~ 15600 5650
+Wire Wire Line
+	15600 3800 15600 5650
+Wire Wire Line
+	15600 5650 15600 7500
+Wire Wire Line
+	15350 7200 15350 5450
+Wire Wire Line
+	15700 5850 15700 7700
+Wire Wire Line
+	15800 5850 15700 5850
+Wire Wire Line
+	15500 5550 15800 5550
+Wire Wire Line
+	15800 5350 15350 5350
+Wire Wire Line
+	15350 5450 15800 5450
+Wire Wire Line
+	15600 5650 15800 5650
+Wire Wire Line
+	15700 5850 15700 4000
+Wire Wire Line
+	15700 4000 15800 4000
+Connection ~ 15700 5850
+$Comp
+L 74xx:74LS00 U?
+U 1 1 611D607C
+P 18100 7500
+F 0 "U?" H 18100 7825 50  0000 C CNN
+F 1 "74LS00" H 18100 7734 50  0000 C CNN
+F 2 "" H 18100 7500 50  0001 C CNN
+F 3 "http://www.ti.com/lit/gpn/sn74ls00" H 18100 7500 50  0001 C CNN
+	1    18100 7500
+	1    0    0    -1
+$EndComp
+Wire Wire Line
+	16800 6900 17100 6900
+Wire Wire Line
+	17100 6900 17100 7600
+Wire Wire Line
+	17100 7600 17800 7600
+Wire Wire Line
+	16800 4950 17200 4950
+Wire Wire Line
+	17200 4950 17200 7400
+Wire Wire Line
+	17200 7400 17800 7400
+Wire Wire Line
+	18400 7500 18400 8450
+Wire Wire Line
+	18400 8450 15700 8450
+Wire Wire Line
+	15700 8450 15700 7700
+Wire Bus Line
+	3150 800  3150 4750
+Wire Bus Line
+	3150 800  8450 800
+Wire Bus Line
+	4300 2000 10700 2000
+Wire Bus Line
+	6100 2200 10700 2200
+Wire Bus Line
+	10700 2000 14650 2000
+Connection ~ 15700 7700
 $EndSCHEMATC

Commit message: Added some display components
Parts:
- removed U?: 74LS00, symbol 74xx:74LS00
- added U13, U14, U15: 74LS161, symbol 74xx:74LS161
- added U16, U17, U? (x8): 74LS30, symbol 74xx:74LS30
- added U18, U19: 74LS04, symbol 74xx:74LS04
- added U20, U21, U? (x4): 74LS00, symbol 74xx:74LS00
- added unit 2 of U9
- added U? (x2): UM61512A, symbol UM61512A:UM61512A
- gave numbers to parts that had none: 12
Connections:
- net labels added: F0, F1, F2, F3, F4, F5, F6, F7, F8, F9, HSYNC, L0, L1, L10, L2, L3, L4, L5, L6, L7, L8, L9, VSync, Vblank, clk, ~F0, ~F1, ~F2, ~F3, ~F5, ~HBLANK, ~L2, ~L4, ~L5, ~L6, ~L7
- wire segments 56 -> 146
Other:
- moved on the sheet: U9A

Commit message: Started Work on graphics solution
Parts:
- added U35: UM61512A, symbol UM61512A:UM61512A
- added U? (x12): 74LS245, symbol 74xx:74LS245
- gave numbers to parts that had none: 7
Connections:
- net labels added: C0, C1, C10, C11, C12, C13, C14, C15, C2, C3, C4, C5, C6, C7, C8, C9, G0, G1, G10, G11, G12, G13, G14, G15, G2, G3, G4, G5, G6, G7, G8, G9, V0, V1, V10, V11, V12, V13, V14, V15, V2, V3, V4, V5, V6, V7, V8, V9
- wire segments 146 -> 233
Other:
- moved on the sheet: U27, U28

Commit message: Working on Graphics
Parts:
- removed U28, U35: UM61512A, symbol UM61512A:UM61512A
- added U? (x5): 74LS04, symbol 74xx:74LS04
- added U? (x2): UM61512A, symbol UM61512A:UM61512A
- added U? (x4): 74HC245, symbol 74xx:74HC245
Connections:
- net +5V: now also U?.1 (A->B), U?.32 (VCC), U?.32 (VCC)
- net Display FSM/X: now also U?.19 (CE), U?.19 (CE), U?.1, U?.19 (CE), U?.9
- net Display FSM/Y: now also U?.19 (CE), U?.19 (CE), U?.24 (OE), U?.3
- net Display FSM/Z: now also U?.19 (CE), U?.19 (CE), U?.24 (OE), U?.5
- net V0: now also U27.12 (A0), U?.12 (A0), U?.12 (A0)
- net V1: now also U27.11 (A1), U?.11 (A1), U?.11 (A1)
- net V10: now also U27.23 (A10), U?.23 (A10), U?.23 (A10)
- net V11: now also U27.25 (A11), U?.25 (A11), U?.25 (A11)
- net V12: now also U27.4 (A12), U?.4 (A12), U?.4 (A12)
- net V13: now also U27.28 (A13), U?.28 (A13), U?.28 (A13)
- net V14: now also U27.3 (A14), U?.3 (A14), U?.3 (A14)
- net V15: now also U27.31 (A15), U?.31 (A15), U?.31 (A15)
- net V2: now also U27.10 (A2), U?.10 (A2), U?.10 (A2)
- net V3: now also U27.9 (A3), U?.9 (A3), U?.9 (A3)
- net V4: now also U27.8 (A4), U?.8 (A4), U?.8 (A4)
- net V5: now also U27.7 (A5), U?.7 (A5), U?.7 (A5)
- net V6: now also U27.6 (A6), U?.6 (A6), U?.6 (A6)
- net V7: now also U27.5 (A7), U?.5 (A7), U?.5 (A7)
- net V8: now also U27.27 (A8), U?.27 (A8), U?.27 (A8)
- net V9: now also U27.26 (A9), U?.26 (A9), U?.26 (A9)
- net at U?.19 (CE), U?.19 (CE): now also U?.2
- net at U?.19 (CE), U?.19 (CE): now also U?.4
- net at U?.19 (CE), U?.19 (CE): now also U?.6
- net D0: now reaches U27.13 (IO1)
- net D0: now also U?.13 (IO1), U?.13 (IO1), U?.18 (B0), U?.2 (A0)
- net D1: now reaches U27.14 (IO2)
- net D1: now also U?.14 (IO2), U?.14 (IO2), U?.17 (B1), U?.3 (A1)
- net D2: now reaches U27.15 (IO3)
- net D2: now also U?.15 (IO3), U?.15 (IO3), U?.16 (B2), U?.4 (A2)
- net D3: now reaches U27.17 (IO4)
- net D3: now also U?.15 (B3), U?.17 (IO4), U?.17 (IO4), U?.5 (A3)
- net D4: now reaches U27.18 (IO5)
- net D4: now also U?.14 (B4), U?.18 (IO5), U?.18 (IO5), U?.6 (A4)
- net D5: now reaches U27.19 (IO6)
- net D5: now also U?.13 (B5), U?.19 (IO6), U?.19 (IO6), U?.7 (A5)
- net D6: now reaches U27.20 (IO7)
- net D6: now also U?.12 (B6), U?.20 (IO7), U?.20 (IO7), U?.8 (A6)
- net D7: now reaches U27.21 (IO8)
- net D7: now also U?.11 (B7), U?.21 (IO8), U?.21 (IO8), U?.9 (A7)
- new net: U?.19 (CE), U?.8
- new net P0: U?.2 (A0)
- new net P1: U?.3 (A1)
- new net P2: U?.4 (A2)
- new net P3: U?.5 (A3)
- new net P4: U?.6 (A4)
- new net P5: U?.7 (A5)
- new net P6: U?.8 (A6)
- new net P7: U?.9 (A7)
- new net S0: U?.18 (B0)
- new net S1: U?.17 (B1)
- new net S2: U?.16 (B2)
- new net S3: U?.15 (B3)
- new net S4: U?.14 (B4)
- new net S5: U?.13 (B5)
- new net S6: U?.12 (B6)
- new net S7: U?.11 (B7)
Other:
- moved on the sheet: U27
